Commit message: Renovated URDF structure using mesh files

File: sequoia_description/urdf/sequoia.urdf.xacro (robot description, xacro)
@@ -3,289 +3,111 @@
   <xacro:include filename="$(find sequoia_description)/urdf/sequoia_gazebo.urdf.xacro"/>
   <xacro:include filename="$(find sequoia_description)/urdf/sequoia_sensors.urdf.xacro"/>
+  <xacro:property name="half_front_track_width" value="0.6" />
+  <xacro:property name="half_rear_track_width" value="0.6" />
+  <xacro:property name="half_wheelbase" value="1.2" />
+  <xacro:property name="wheel_radius" value="0.32" />
+  <xacro:property name="wheel_thickness" value="0.17" />
+  <xacro:property name="wheel_mass" value="20.0" />
+  <xacro:property name="body_mass" value="1620.0" />
+  <xacro:property name="body_width" value="${2*half_rear_track_width}" />
+  <xacro:property name="body_depth" value="${2*half_wheelbase + 0.8}" />
+  <xacro:property name="body_length" value="0.6" />
+  <xacro:macro name="rear_wheel" params="name x y z flip" >
+    <link name="wheel_${name}" >
+      <visual>
+        <origin xyz="0 0 0" rpy="0 ${flip * pi - pi/2} 0" />
+        <geometry>
+          <mesh filename="package://sequoia_description/meshes/wheel.dae" scale="2.54 2.54 2.54" />
+        </geometry>
+      </visual>
+      <collision>
+        <geometry>
+          <cylinder radius="${wheel_radius}" length="${wheel_thickness}" />
+        </geometry>
+      </collision>
+      <inertial>
+        <origin xyz="0 0 0" rpy="0 0 0"/>
+        <mass value="${wheel_mass}"/>
+        <inertia ixx="${wheel_mass/12*(3*wheel_radius*wheel_radius + wheel_thickness*wheel_thickness)}" ixy="0" ixz="0" iyy="${wheel_mass/12*(3*wheel_radius*wheel_radius + wheel_thickness*wheel_thickness)}" iyz="0" izz="${wheel_mass/2 * wheel_radius*wheel_radius}"/>
+      </inertial>
+    </link>
+    <joint name="wheel_${name}" type="continuous" >
+      <parent link="base_link" />
+      <child link="wheel_${name}" />
+      <origin xyz="${x} ${y} ${z}" rpy="-1.57079632679 0 0" />
+      <axis xyz="0 0 1" />
+      <limit effort="1000.0" velocity="22.0" />
+    </joint>
+  </xacro:macro>
+  <xacro:macro name="front_wheel" params="name x y z flip" >
+    <link name="wheel_${name}" >
+      <visual>
+        <origin xyz="0 0 0" rpy="0 ${flip * pi - pi/2} 0" />
+        <geometry>
+          <mesh filename="package://sequoia_description/meshes/wheel.dae" scale="2.54 2.54 2.54" />
+        </geometry>
+      </visual>
+      <collision>
+        <geometry>
+          <cylinder radius="${wheel_radius}" length="${wheel_thickness}" />
+        </geometry>
+      </collision>
+      <inertial>
+        <origin xyz="0 0 0" rpy="0 0 0"/>
+        <mass value="${wheel_mass}"/>
+        <inertia ixx="${wheel_mass/12*(3*wheel_radius*wheel_radius + wheel_thickness*wheel_thickness)}" ixy="0" ixz="0" iyy="${wheel_mass/12*(3*wheel_radius*wheel_radius + wheel_thickness*wheel_thickness)}" iyz="0" izz="${wheel_mass/2 * wheel_radius*wheel_radius}"/>
+      </inertial>
+    </link>
+    <link name="steer_${name}" >
+      <inertial>
+        <origin xyz="0 0 0" rpy="0 0 0"/>
+        <mass value="20.0"/>
+        <inertia ixx="0.1" ixy="0" ixz="0" iyy="0.1" iyz="0" izz="0.1"/>
+      </inertial>
+    </link>
+    <joint name="steer_${name}" type="revolute" >
+      <parent link="base_link" />
+      <child link="steer_${name}" />
+      <origin xyz="${x} ${y} ${z}" rpy="0 0 0" />
+      <axis xyz="0 0 1" />
+      <limit upper="0.6" lower="-0.6" effort="0.0" velocity="0.0" />
+    </joint>
+    <joint name="wheel_${name}" type="continuous" >
+      <parent link="steer_${name}" />
+      <child link="wheel_${name}" />
+      <origin xyz="0 0 0" rpy="-1.57079632679 0 0" />
+      <axis xyz="0 0 1" />
+      <limit effort="1000.0" velocity="22.0" />
+    </joint>
+  </xacro:macro>
   <link name="base_footprint">
-  </link>
-  <link name="rearaxle">
-  </link>
-  <link name="frontaxle">
   </link>
   <link name="base_link">
     <inertial>
-      <origin xyz="0 0 0" rpy="0 0 0"/>
-      <mass value="900.0"/>
-      <inertia ixx="1000.0" ixy="0" ixz="0" iyy="1000.0" iyz="0" izz="1000.0"/>
+      <origin xyz="0 0 0.75" rpy="0 0 0"/>
+      <mass value="${body_mass}"/>
+      <inertia ixx="${body_mass/12 * (body_width*body_width + body_length*body_length)}" ixy="0" ixz="0" iyy="${body_mass/12 * (body_length*body_length + body_depth*body_depth)}" iyz="0" izz="${body_mass/12 * (body_width*body_width + body_depth*body_depth)}"/>
     </inertial>
-    <visual name="base_link_visual">
-      <origin xyz="-0.0 0 0.0" rpy="0 0 0"/>
+    <visual>
+      <origin xyz="-0.22 0 0.07" rpy="0 0 0"/>
       <geometry>
-        <box size="2.3241 1.3516 0.635"/>
+        <mesh filename="package://sequoia_description/meshes/body.dae" scale="1 1 1" />
       </geometry>
-      <material name="white"/>
     </visual>
-    <collision name="base_link_collision">
-      <origin xyz="0 0 0" rpy="0 0 0"/>
+    <collision>
+      <origin xyz="-0.22 0 0.07" rpy="0 0 0"/>
       <geometry>
-        <box size="2.3241 1.3516 0.635"/>
+        <mesh filename="package://sequoia_description/meshes/body_collision.stl" scale="1 1 1" />
       </geometry>
     </collision>
   </link>
-  <link name="front_end">
-    <inertial>
-      <origin xyz="0 0 0" rpy="0 0 0"/>
-      <mass value="100.0"/>
-      <inertia ixx="1000.0" ixy="0" ixz="0" iyy="1000.0" iyz="0" izz="1000.0"/>
-    </inertial>
-    <visual name="front_end_visual">
-      <origin xyz="-0.0 0 0.0" rpy="0 0 0"/>
-      <geometry>
-        <cylinder radius="0.3175" length="1.3516"/>
-      </geometry>
-      <material name="white"/>
-    </visual>
-    <collision name="front_end_collision">
-      <origin xyz="-0.0 0 0.0" rpy="0 0 0"/>
-      <geometry>
-        <cylinder radius="0.3175" length="1.3516"/>
-      </geometry>
-    </collision>
-  </link>
-  <link name="trunk">
-    <inertial>
-      <origin xyz="0 0 0" rpy="0 0 0"/>
-      <mass value="20.0"/>
-      <inertia ixx="1000.0" ixy="0" ixz="0" iyy="1000.0" iyz="0" izz="1000.0"/>
-    </inertial>
-    <visual name="trunk_visual">
-      <origin xyz="-0.0 0 0.0" rpy="0 0 0"/>
-      <geometry>
-        <box size="0.5 1.2 0.4"/>
-      </geometry>
-      <material name="white"/>
-    </visual>
-    <collision name="trunk_collision">
-      <origin xyz="0 0 0" rpy="0 0 0"/>
-      <geometry>
-        <box size="0.5 1.2 0.4"/>
-      </geometry>
-    </collision>
-  </link>
-  <link name="dome">
-    <inertial>
-      <origin xyz="0 0 0" rpy="0 0 0"/>
-      <mass value="200.0"/>
-      <inertia ixx="1000.0" ixy="0" ixz="0" iyy="1000.0" iyz="0" izz="1000.0"/>
-    </inertial>
-    <visual name="dome_visual">
-      <origin xyz="-0.0 0 0.0" rpy="0 0 0"/>
-      <geometry>
-        <cylinder radius="0.8"  length="1.350"/>
-      </geometry>
-      <material name="grey"/>
-    </visual>
-    <collision name="dome_collision">
-      <origin xyz="0 0 0" rpy="0 0 0"/>
-      <geometry>
-        <cylinder radius="0.8"  length="1.350"/>
-      </geometry>
-    </collision>
-  </link>
-  <link name="dome_small">
-    <inertial>
-      <origin xyz="0 0 0" rpy="0 0 0"/>
-      <mass value="1.0"/>
-      <inertia ixx="1000.0" ixy="0" ixz="0" iyy="1000.0" iyz="0" izz="1000.0"/>
-    </inertial>
-    <visual name="dome_small_visual">
-      <origin xyz="-0.0 0 0.0" rpy="0 0 0"/>
-      <geometry>
-        <cylinder radius="0.2"  length="1.345"/>
-      </geometry>
-      <material name="black"/>
-    </visual>
-    <collision name="dome_small_collision">
-      <origin xyz="0 0 0" rpy="0 0 0"/>
-      <geometry>
-        <cylinder radius="0.2"  length="1.345"/>
-      </geometry>
-    </collision>
-  </link>
-  <link name="left_steer">
-    <inertial>
-      <origin xyz="0 0 0" rpy="0 0 0"/>
-      <mass value="10.0"/>
-      <inertia ixx="0.37" ixy="0" ixz="0" iyy="0.4" iyz="0" izz="0.6"/>
-    </inertial>
-  </link>
-  <link name="right_steer">
-    <inertial>
-      <origin xyz="0 0 0" rpy="0 0 0"/>
-      <mass value="10.0"/>
-      <inertia ixx="0.37" ixy="0" ixz="0" iyy="0.4" iyz="0" izz="0.6"/>
-    </inertial>
-  </link>
-  <link name="wheel_fl">
-    <inertial>
-      <origin xyz="0 0 0" rpy="0 0 0"/>
-      <mass value="0.75"/>
-      <inertia ixx="0.305" ixy="0" ixz="0" iyy="0.305" iyz="0" izz="0.5445"/>
-    </inertial>
-    <visual name="wheel_fl_visual">
-      <origin xyz="-0.0 0 0" rpy="-3.141593 0 0"/>
-      <geometry>
-        <cylinder radius="0.254" length="0.127"/>
-      </geometry>
-      <material name="Tire_001.004"/>
-    </visual>
-    <collision name="wheel_fl_collision">
-      <origin xyz="-0.0 0 0" rpy="-3.141593 0 0"/>
-      <geometry>
-        <cylinder radius="0.254" length="0.127"/>
-      </geometry>
-    </collision>
-  </link>
-  <link name="wheel_fr">
-    <inertial>
-      <origin xyz="0.0 0 0" rpy="0 0 0"/>
-      <mass value="0.75"/>
-      <inertia ixx="0.305" ixy="0" ixz="0" iyy="0.305" iyz="0" izz="0.5445"/>
-    </inertial>
-    <visual name="wheel_fr_visual">
-      <origin xyz="-0.0 0 0" rpy="-3.141593 0 0"/>
-      <geometry>
-        <cylinder radius="0.254" length="0.127"/>
-      </geometry>
-      <material name="Tire_001.006"/>
-    </visual>
-    <collision name="wheel_fr_collision">
-      <origin xyz="0 0 0" rpy="-3.141593 0 0"/>
-      <geometry>
-        <cylinder radius="0.254" length="0.127"/>
-      </geometry>
-    </collision>
-  </link>
-  <link name="wheel_rl">
-    <inertial>
-      <origin xyz="0.00 0 0" rpy="0 0 0"/>
-      <mass value="0.75"/>
-      <inertia ixx="0.305" ixy="0" ixz="0" iyy="0.305" iyz="0" izz="0.5445"/>
-    </inertial>
-    <visual name="wheel_rl_visual">
-      <origin xyz="-0.0 0 0" rpy="-3.141593 0 0"/>
-      <geometry>
-        <cylinder radius="0.254" length="0.127"/>
-      </geometry>
-      <material name="Tire_001.005"/>
-    </visual>
-    <collision name="wheel_rl_collision">
-      <origin xyz="-0.00 0 0" rpy="-3.141593 0 0"/>
-      <geometry>
-      <cylinder radius="0.254" length="0.127"/>
-      </geometry>
-    </collision>
-  </link>
-  <link name="wheel_rr">
-    <inertial>
-      <origin xyz="0.00 0 0" rpy="0 0 0"/>
-      <mass value="0.75"/>
-      <inertia ixx="0.305" ixy="0" ixz="0" iyy="0.305" iyz="0" izz="0.5445"/>
-    </inertial>
-    <visual name="wheel_rr_visual">
-      <origin xyz="-0.0 0 0" rpy="-3.141593 0 0"/>
-      <geometry>
-        <cylinder radius="0.254" length="0.127"/>
-      </geometry>
-      <material name="Tire_001.007"/>
-    </visual>
-    <collision name="wheel_rr_collision">
-      <origin xyz="0.00 0 0" rpy="-3.141593 0 0"/>
-      <geometry>
-      <cylinder radius="0.254" length="0.127"/>
-      </geometry>
-    </collision>
-  </link>
-  <joint name="rearaxle" type="fixed">
-    <origin xyz="-0.9668 0 0.0" rpy="0 0 0"/>
-    <parent link="base_footprint"/>
-    <child link="rearaxle"/>
-  </joint>
-  <joint name="frontaxle" type="fixed">
-    <origin xyz="0.9668 0 0.0" rpy="0 0 0"/>
-    <parent link="base_footprint"/>
-    <child link="frontaxle"/>
-  </joint>
+  <xacro:rear_wheel name="rl" x="${-half_wheelbase}" y="${half_rear_track_width}" z="0" flip="1" />
+  <xacro:rear_wheel name="rr" x="${-half_wheelbase}" y="${-half_rear_track_width}" z="0" flip="0" />
+  <xacro:front_wheel name="fl" x="${half_wheelbase}" y="${half_front_track_width}" z="0" flip="1" />
+  <xacro:front_wheel name="fr" x="${half_wheelbase}" y="${-half_front_track_width}" z="0" flip="0" />
   <joint name="base_link" type="fixed">
-    <origin xyz="-0.15875 0 0.508" rpy="0 0 0"/>
+    <origin xyz="${half_wheelbase} 0 ${wheel_radius}" rpy="0 0 0"/>
     <parent link="base_footprint"/>
     <child link="base_link"/>
   </joint>
-  <joint name="front_end" type="fixed">
-    <origin xyz="1.0033 0 0.508" rpy="-1.570796 0 0"/>
-    <parent link="base_footprint"/>
-    <child link="front_end"/>
-  </joint>
-  <joint name="dome" type="fixed">
-    <origin xyz="-0.1 0 1.258" rpy="-1.570796 0 0"/>
-    <parent link="base_footprint"/>
-    <child link="dome"/>
-  </joint>
-  <joint name="dome_small" type="fixed">
-    <origin xyz="0.7 0 0.9" rpy="-1.570796 0 0"/>
-    <parent link="base_footprint"/>
-    <child link="dome_small"/>
-  </joint>
-  <joint name="trunk" type="fixed">
-    <origin xyz="-1.05 0 1.1" rpy="0 -0.1 0.0"/>
-    <parent link="base_footprint"/>
-    <child link="trunk"/>
-  </joint>
-  <joint name="left_steer" type="revolute">
-    <origin xyz="1.12555 0.6258 -0.254" rpy="0 0 0"/>
-    <parent link="base_link"/>
-    <child link="left_steer"/>
-    <axis xyz="0 0 1.0"/>
-    <limit lower="-0.7" upper="0.7" effort="500000.0" velocity="100.0"/>
-  </joint>
-  <joint name="right_steer" type="revolute">
-    <origin xyz="1.12555 -0.6258 -0.254" rpy="0 0 0"/>
-    <parent link="base_link"/>
-    <child link="right_steer"/>
-    <axis xyz="0 0 1.0"/>
-    <limit lower="-0.7" upper="0.7" effort="500000.0" velocity="100.0"/>
-  </joint>
-  <joint name="wheel_fl" type="continuous">
-    <origin xyz="0.0 0.0 0.0" rpy="-1.570796 0 0"/>
-    <parent link="left_steer"/>
-    <child link="wheel_fl"/>
-    <axis xyz="0 0 1.0"/>
-    <limit effort="5000.0" velocity="2.235"/>
-  </joint>
-  <joint name="wheel_fr" type="continuous">
-    <origin xyz="0 0 0" rpy="-1.570796 0 0"/>
-    <parent link="right_steer"/>
-    <child link="wheel_fr"/>
-    <axis xyz="0 0 1.0"/>
-    <limit effort="5000.0" velocity="2.235"/>
-  </joint>
-  <joint name="wheel_rl" type="continuous">
-    <origin xyz="-0.80805 0.6258 -0.254" rpy="-1.570796 0 0"/>
-    <parent link="base_link"/>
-    <child link="wheel_rl"/>
-    <axis xyz="0 0 1.0"/>
-    <limit effort="10000.0" velocity="2.235"/>
-  </joint>
-  <joint name="wheel_rr" type="continuous">
-    <origin xyz="-0.80805 -0.6258 -0.254" rpy="-1.570796 0 0"/>
-    <parent link="base_link"/>
-    <child link="wheel_rr"/>
-    <axis xyz="0 0 1.0"/>
-    <limit effort="10000.0" velocity="2.235"/>
-  </joint>
-  <material name="white">
-    <color rgba="1 1 1 1"/>
-  </material>
-  <material name="grey">
-    <color rgba="0.5 0.5 0.5 1" />
-  </material>
-  <material name="black">
-    <color rgba="0.2 0.2 0.2 1" />
-  </material>
 </robot>

File: sequoia_description/urdf/sequoia_gazebo.urdf.xacro (robot description, xacro)
@@ -8,5 +8,5 @@
     <plugin name="joint_state_publisher" filename="libgazebo_ros_joint_state_publisher.so">
       <jointName>
-          left_steer, right_steer, wheel_fl, wheel_fr, wheel_rl, wheel_rr
+          steer_fl, steer_fr, wheel_fl, wheel_fr, wheel_rl, wheel_rr
       </jointName>
       <updateRate>100</updateRate>
@@ -18,10 +18,4 @@
     <mu1>0.5</mu1>
     <mu2>0.5</mu2>
-  </gazebo>
-  <gazebo reference="dome" >
-    <material>Gazebo/Grey</material>
-  </gazebo>
-  <gazebo reference="dome_small" >
-    <material>Gazebo/Black</material>
   </gazebo>
   <gazebo reference="wheel_fl" >

File: sequoia_description/urdf/sequoia_sensors.urdf.xacro (robot description, xacro)
@@ -3,10 +3,10 @@
   <!-- Camera -->
   <xacro:include filename="$(find sequoia_description)/urdf/sensors/camera.urdf.xacro" />
-  <xacro:camera_sim name="camera_sim" parent_link="base_footprint" x="0.45" y="0" z="1.9" roll="0" pitch="0.4" yaw="0" />
+  <xacro:camera_sim name="camera_sim" parent_link="base_footprint" x="1.65" y="0" z="2.1" roll="0" pitch="0.4" yaw="0" />
   <!-- LIDAR -->
   <xacro:include filename="$(find sequoia_description)/urdf/sensors/hokuyo_utm_30.urdf.xacro" />
-  <xacro:hokuyo_utm_30 name="laser" parent_frame="base_footprint" x="1.2" y="0.0" z="0.85" roll="0.0" pitch="0.0" yaw="0.0" />
+  <xacro:hokuyo_utm_30 name="laser" parent_frame="base_footprint" x="2.75" y="0.0" z="0.85" roll="0.0" pitch="0.0" yaw="0.0" />
   <!-- GPS -->
   <xacro:include filename="$(find sequoia_description)/urdf/sensors/gps.urdf.xacro" />
-  <xacro:gps name="gps" parent_frame="base_footprint" x="0" y="0" z="2.06" />
+  <xacro:gps name="gps" parent_frame="base_footprint" x="0.8" y="0" z="2.35" />
 </robot>

Commit message: Created Gazebo plugin to simulate the vehicle interface
Interface is similar to the old version of the simulator. The interface should change to be the same as the real vehicle.

File: sequoia_description/urdf/sequoia.urdf.xacro (robot description, xacro)
@@ -8,6 +8,6 @@
   <xacro:property name="wheel_radius" value="0.32" />
   <xacro:property name="wheel_thickness" value="0.17" />
-  <xacro:property name="wheel_mass" value="20.0" />
-  <xacro:property name="body_mass" value="1620.0" />
+  <xacro:property name="wheel_mass" value="10.0" />
+  <xacro:property name="body_mass" value="544.0" />
   <xacro:property name="body_width" value="${2*half_rear_track_width}" />
   <xacro:property name="body_depth" value="${2*half_wheelbase + 0.8}" />

File: sequoia_description/urdf/sequoia_gazebo.urdf.xacro (robot description, xacro)
@@ -3,5 +3,5 @@
   <gazebo>
     <!-- Simulated vehicle interface -->
-    <plugin name="gembot_interface_plugin" filename="libgembot_interface_plugin.so" >
+    <plugin name="sequoia_interface" filename="libsequoia_interface_plugin.so" >
     </plugin>
     <!-- Publish JointState message -->

Commit message: Initial calibration of lane detection camera; tested 3D pixel projection

File: sequoia_description/urdf/sequoia.urdf.xacro (robot description, xacro)
@@ -2,5 +2,30 @@
 <robot name="sequoia" xmlns:xacro="http://www.ros.org/wiki/xacro">
   <xacro:include filename="$(find sequoia_description)/urdf/sequoia_gazebo.urdf.xacro"/>
-  <xacro:include filename="$(find sequoia_description)/urdf/sequoia_sensors.urdf.xacro"/>
+  <xacro:unless value="$(arg live)" >
+    <xacro:include filename="$(find sequoia_description)/urdf/sequoia_sensors.urdf.xacro"/>
+  </xacro:unless>
+  <xacro:if value="$(arg live)" >
+    <link name="lane_camera" >
+      <visual>
+        <geometry>
+          <box size="0.1 0.1 0.1" />
+        </geometry>
+        <material name="white">
+          <color rgba="1 1 1 1" />
+        </material>
+      </visual>
+    </link>
+    <link name="lane_camera_optical" />
+    <joint name="lane_camera_optical" type="fixed" >
+      <parent link="lane_camera_optical" />
+      <child link="lane_camera" />
+      <origin xyz="0 0 0" rpy="-1.57079632679 0 -1.57079632679" />
+    </joint>
+    <joint name="camera_mount" type="fixed" >
+      <parent link="base_footprint" />
+      <child link="lane_camera_optical" />
+      <origin xyz="1.613 0 1.473" rpy="0 0.539 0" />
+    </joint>
+  </xacro:if>
   <xacro:property name="half_front_track_width" value="0.6" />
   <xacro:property name="half_rear_track_width" value="0.6" />

Commit message: Added live GPS antenna TF frame to URDF model

File: sequoia_description/urdf/sequoia.urdf.xacro (robot description, xacro)
@@ -26,4 +26,19 @@
       <child link="lane_camera_optical" />
       <origin xyz="1.613 0 1.473" rpy="0 0.539 0" />
+    </joint>
+    <link name="gps_antenna" >
+      <visual>
+        <geometry>
+          <cylinder radius="0.1" length="0.1" />
+        </geometry>
+        <material name="white">
+          <color rgba="1 1 1 1" />
+        </material>
+      </visual>
+    </link>
+    <joint name="gps_antenna" type="fixed" >
+      <parent link="base_footprint" />
+      <child link="gps_antenna" />
+      <origin xyz="0.711 -0.559 1.905" rpy="0 0 0" />
     </joint>
   </xacro:if>

Commit message: Updated calibration of real lane camera in URDF model

File: sequoia_description/urdf/sequoia.urdf.xacro (robot description, xacro)
@@ -25,5 +25,5 @@
       <parent link="base_footprint" />
       <child link="lane_camera_optical" />
-      <origin xyz="1.613 0 1.473" rpy="0 0.539 0" />
+      <origin xyz="1.435 0 1.6" rpy="0 0.68 0" />
     </joint>
     <link name="gps_antenna" >

Commit message: Added LIDAR frame to URDF model

File: sequoia_description/urdf/sequoia.urdf.xacro (robot description, xacro)
@@ -41,4 +41,19 @@
       <child link="gps_antenna" />
       <origin xyz="0.711 -0.559 1.905" rpy="0 0 0" />
+    </joint>
+    <link name="laser" >
+      <visual>
+        <geometry>
+          <box size="0.1 0.1 0.1" />
+        </geometry>
+        <material name="white">
+          <color rgba="1 1 1 1" />
+        </material>
+      </visual>
+    </link>
+    <joint name="laser" type="fixed" >
+      <parent link="base_footprint" />
+      <child link="laser" />
+      <origin xyz="2.28 0 0" rpy="0 0 0" />
     </joint>
   </xacro:if>
